File: UccMicroDuino.kicad_sch (KiCad schematic)
At the start: 8 parts, among them J2 Conn_01x10_Socket, J2 USB_A, U2 ATtiny85-20S

Commit message: Mi primer cambio para el practico 2
Parts:
- added D3: 3.6V 1/2 mW, Diode_SMD:D_SOD-123, symbol Device:D_Zener
- added D4: Led green, ledSmd:ledSMD, symbol Device:LED
- added R2: R, symbol Device:R
- added R2, R3: 68Ω 5% 1/8W, symbol Device:R
- added R4: 330Ω 5% 1/8W, symbol Device:R
- D2: renamed from D1; value D_Zener -> 3.6V 1/2 mW
- J1: renamed from J2; value USB_A -> Pcb USB type A
- J2: value Conn_01x10_Socket -> Header
- R1: value R -> 1.5KΩ 5% 1/8W
- renumbered D5 to D1, U2 to U1
Connections:
- net +5V: now also C1.1, D3.2 (A), J2.1 (Pin_1), U1.8 (VCC)
- net GND: now also C1.2, D2.2 (A), J1.4 (GND), J2.2 (Pin_2), U1.4 (GND), D3.2 (A), R2.2, R4.1
- net at D3.1 (K): now also R2.1
- net at R1.2: now also D2.1 (K), J1.2 (D-), R2.2
- net at U1.1 (~{RESET}/PB5): now also J2.9 (Pin_9)
- net at U1.2 (XTAL1/PB3): now also J2.7 (Pin_7), R2.1
- net at U1.3 (XTAL2/PB4): now also J2.8 (Pin_8), R3.1
- net at U1.5 (AREF/PB0): now also J2.4 (Pin_4)
- net at U1.6 (PB1): now also J2.5 (Pin_5), D4.2 (A)
- net at U1.7 (PB2): now also J2.6 (Pin_6)
- net at J1.1 (VBUS): now also D1.2 (A)
- net at J1.3 (D+): now also D3.1 (K), R3.2
- new net: D4.1 (K), R4.2
- no-connect marks 0 -> 2
Other:
- moved on the sheet: D3, U1
